File: kicad/ent/ent.sch (KiCad schematic (older format))
At the start: 16 parts

Commit message: updated schema
Parts:
- added C5: 100nF, symbol Device:C
- added J1, J3: Conn_01x04_Male, symbol Connector:Conn_01x04_Male
- added J2: Conn_01x12_Male, symbol Connector:Conn_01x12_Male
- added J4: Conn_01x06_Male, symbol Connector:Conn_01x06_Male
- added R2, R3: 10k, symbol Device:R
- added SW1: SW_SPDT, symbol Switch:SW_SPDT
- added SW2: SW_Push, symbol Switch:SW_Push
- P1, P2, P3: renamed from P?; symbol ian:mesure_pad -> ent-rescue:mesure_pad-ian
- U2: renamed from U?; symbol ian:LIS2DHTR -> ent-rescue:LIS2DHTR-ian
- gave numbers to parts that had none: 12
Connections:
- net labels added: INT1, INT2, NSS1, NSS2, NSS3, NSS4, SPI1_MISO, SPI1_MOSI, SPI1_SCK, STOP1, STOP2, STOP3, STOP4, SWCLK, SWDIO
- net labels removed: GNDPWR
- wire segments 84 -> 99
- no-connect marks 0 -> 7

Commit message: schema main done
Parts:
- removed J4: Conn_01x06_Male, symbol Connector:Conn_01x06_Male
- removed P1, P2, P3: mesure_pad, symbol ent-rescue:mesure_pad-ian
- added J4, J5, J6, J7: Conn_01x03_Male, Connector_JST:JST_XH_B3B-XH-A_1x03_P2.50mm_Vertical, symbol Connector:Conn_01x03_Male
- added TP1, TP2, TP3: TestPoint, TestPoint:TestPoint_Pad_D2.0mm, symbol Connector:TestPoint
- C1, C2, C3, C4, C5, C6, C7, C8: footprint (none) -> Capacitor_SMD:C_0805_2012Metric_Pad1.15x1.40mm_HandSolder
- J1, J3: footprint (none) -> Connector_JST:JST_XH_B4B-XH-A_1x04_P2.50mm_Vertical
- J2: footprint (none) -> Connector_JST:JST_XH_B12B-XH-A_1x12_P2.50mm_Vertical
- L1: footprint (none) -> Inductor_SMD:L_0805_2012Metric_Pad1.15x1.40mm_HandSolder
- R1, R2, R3, R4: footprint (none) -> Resistor_SMD:R_0805_2012Metric_Pad1.15x1.40mm_HandSolder
- SW1: footprint (none) -> Connector_PinHeader_2.54mm:PinHeader_1x03_P2.54mm_Vertical
- SW2: footprint (none) -> Button_Switch_SMD:SW_SPST_PTS645
Connections:
- net +3V3: now also J4.3 (Pin_3), J5.3 (Pin_3), J6.3 (Pin_3), J7.3 (Pin_3), TP2.1
- net GND: now also J4.1 (Pin_1), J5.1 (Pin_1), J6.1 (Pin_1), J7.1 (Pin_1), TP3.1
- net STOP1: now also J4.2 (Pin_2)
- net STOP2: now also J6.2 (Pin_2)
- net STOP3: now also J5.2 (Pin_2)
- net STOP4: now also J7.2 (Pin_2)
- net at R1.1, U1.8 (PG): now also TP1.1

Commit message: + motor drivers
Parts:
- renumbered J4 to J2, J5 to J3, J2 to J4, J3 to J5
Changed lines of the file:
@@
 EESchema Schematic File Version 4
-LIBS:ent-cache
-EELAYER 29 0
+EELAYER 30 0
 EELAYER END
 $Descr A4 11693 8268
@@
 $EndComp
 $Comp
-L power:GND #PWR022
+L power:GND #PWR026
 U 1 1 5E464C89
 P 8250 1750
-F 0 "#PWR022" H 8250 1500 50  0001 C CNN
+F 0 "#PWR026" H 8250 1500 50  0001 C CNN
 F 1 "GND" H 8255 1577 50  0000 C CNN
 F 2 "" H 8250 1750 50  0001 C CNN
@@
 $EndComp
 $Comp
-L power:+3V3 #PWR021
+L power:+3V3 #PWR025
 U 1 1 5E465814
 P 8250 950
-F 0 "#PWR021" H 8250 800 50  0001 C CNN
+F 0 "#PWR025" H 8250 800 50  0001 C CNN
 F 1 "+3V3" H 8265 1123 50  0000 C CNN
 F 2 "" H 8250 950 50  0001 C CNN
@@
 $EndComp
 $Comp
-L power:GND #PWR026
+L power:GND #PWR030
 U 1 1 5E50BF14
 P 8800 3000
-F 0 "#PWR026" H 8800 2750 50  0001 C CNN
+F 0 "#PWR030" H 8800 2750 50  0001 C CNN
 F 1 "GND" H 8805 2827 50  0000 C CNN
 F 2 "" H 8800 3000 50  0001 C CNN
@@
 $EndComp
 $Comp
-L power:GND #PWR024
+L power:GND #PWR028
 U 1 1 5E597546
 P 8800 2000
-F 0 "#PWR024" H 8800 1750 50  0001 C CNN
+F 0 "#PWR028" H 8800 1750 50  0001 C CNN
 F 1 "GND" V 8805 1827 50  0000 C CNN
 F 2 "" H 8800 2000 50  0001 C CNN
@@
 $EndComp
 $Comp
-L power:+12V #PWR023
+L power:+12V #PWR027
 U 1 1 5E598788
 P 8800 1900
-F 0 "#PWR023" H 8800 1750 50  0001 C CNN
+F 0 "#PWR027" H 8800 1750 50  0001 C CNN
 F 1 "+12V" H 8815 2073 50  0000 C CNN
 F 2 "" H 8800 1900 50  0001 C CNN
@@
 	6400 3600 6700 3600
 $Comp
-L Connector:Conn_01x04_Male J3
+L Connector:Conn_01x04_Male J5
 U 1 1 5E5B5B5B
 P 9000 3650
-F 0 "J3" H 8972 3532 50  0000 R CNN
+F 0 "J5" H 8972 3532 50  0000 R CNN
 F 1 "Conn_01x04_Male" H 8972 3623 50  0000 R CNN
 F 2 "Connector_JST:JST_XH_B4B-XH-A_1x04_P2.50mm_Vertical" H 9000 3650 50  0001 C CNN
@@
 SWDIO
 $Comp
-L power:GND #PWR028
+L power:GND #PWR032
 U 1 1 5E5B738E
 P 8800 3750
-F 0 "#PWR028" H 8800 3500 50  0001 C CNN
+F 0 "#PWR032" H 8800 3500 50  0001 C CNN
 F 1 "GND" H 8805 3577 50  0000 C CNN
 F 2 "" H 8800 3750 50  0001 C CNN
@@
 $EndComp
 $Comp
-L power:+3V3 #PWR027
+L power:+3V3 #PWR031
 U 1 1 5E5B7E1D
 P 8800 3450
-F 0 "#PWR027" H 8800 3300 50  0001 C CNN
+F 0 "#PWR031" H 8800 3300 50  0001 C CNN
 F 1 "+3V3" H 8815 3623 50  0000 C CNN
 F 2 "" H 8800 3450 50  0001 C CNN
@@
 $EndComp
 $Comp
-L Connector:Conn_01x12_Male J2
+L Connector:Conn_01x12_Male J4
 U 1 1 5E5BE1AD
 P 9000 2500
-F 0 "J2" H 8972 2382 50  0000 R CNN
+F 0 "J4" H 8972 2382 50  0000 R CNN
 F 1 "Conn_01x12_Male" H 8972 2473 50  0000 R CNN
 F 2 "Connector_JST:JST_XH_B12B-XH-A_1x12_P2.50mm_Vertical" H 9000 2500 50  0001 C CNN
@@
 INT2
 $Comp
-L power:+3V3 #PWR025
+L power:+3V3 #PWR029
 U 1 1 5E61BC89
 P 8800 2100
-F 0 "#PWR025" H 8800 1950 50  0001 C CNN
+F 0 "#PWR029" H 8800 1950 50  0001 C CNN
 F 1 "+3V3" V 8815 2228 50  0000 L CNN
 F 2 "" H 8800 2100 50  0001 C CNN
@@
 $EndComp
 $Comp
-L power:+3.3V #PWR0101
+L power:+3.3V #PWR033
 U 1 1 5E656DEC
 P 9400 4250
-F 0 "#PWR0101" H 9400 4100 50  0001 C CNN
+F 0 "#PWR033" H 9400 4100 50  0001 C CNN
 F 1 "+3.3V" H 9415 4423 50  0000 C CNN
 F 2 "" H 9400 4250 50  0001 C CNN
@@
 $EndComp
 $Comp
-L power:GND #PWR0102
+L power:GND #PWR034
 U 1 1 5E65891B
 P 9400 4450
-F 0 "#PWR0102" H 9400 4200 50  0001 C CNN
+F 0 "#PWR034" H 9400 4200 50  0001 C CNN
 F 1 "GND" H 9405 4277 50  0000 C CNN
 F 2 "" H 9400 4450 50  0001 C CNN
@@
 $EndComp
 $Comp
-L power:+3.3V #PWR0103
+L power:+3.3V #PWR035
 U 1 1 5E667123
 P 9400 4900
-F 0 "#PWR0103" H 9400 4750 50  0001 C CNN
+F 0 "#PWR035" H 9400 4750 50  0001 C CNN
 F 1 "+3.3V" H 9415 5073 50  0000 C CNN
 F 2 "" H 9400 4900 50  0001 C CNN
@@
 $EndComp
 $Comp
-L power:GND #PWR0104
+L power:GND #PWR036
 U 1 1 5E667129
 P 9400 5100
-F 0 "#PWR0104" H 9400 4850 50  0001 C CNN
+F 0 "#PWR036" H 9400 4850 50  0001 C CNN
 F 1 "GND" H 9405 4927 50  0000 C CNN
 F 2 "" H 9400 5100 50  0001 C CNN
@@
 STOP1
 $Comp
-L Connector:Conn_01x03_Male J4
+L Connector:Conn_01x03_Male J2
 U 1 1 5E66BEE7
 P 8300 4350
-F 0 "J4" H 8272 4282 50  0000 R CNN
+F 0 "J2" H 8272 4282 50  0000 R CNN
 F 1 "Conn_01x03_Male" H 8272 4373 50  0000 R CNN
 F 2 "Connector_JST:JST_XH_B3B-XH-A_1x03_P2.50mm_Vertical" H 8300 4350 50  0001 C CNN
@@
 $EndComp
 $Comp
-L power:+3.3V #PWR0105
+L power:+3.3V #PWR021
 U 1 1 5E66BEED
 P 8100 4250
-F 0 "#PWR0105" H 8100 4100 50  0001 C CNN
+F 0 "#PWR021" H 8100 4100 50  0001 C CNN
 F 1 "+3.3V" H 8115 4423 50  0000 C CNN
 F 2 "" H 8100 4250 50  0001 C CNN
@@
 $EndComp
 $Comp
-L power:GND #PWR0106
+L power:GND #PWR022
 U 1 1 5E66BEF3
 P 8100 4450
-F 0 "#PWR0106" H 8100 4200 50  0001 C CNN
+F 0 "#PWR022" H 8100 4200 50  0001 C CNN
 F 1 "GND" H 8105 4277 50  0000 C CNN
 F 2 "" H 8100 4450 50  0001 C CNN
@@
 STOP3
 $Comp
-L Connector:Conn_01x03_Male J5
+L Connector:Conn_01x03_Male J3
 U 1 1 5E66EF9D
 P 8300 5050
-F 0 "J5" H 8272 4982 50  0000 R CNN
+F 0 "J3" H 8272 4982 50  0000 R CNN
 F 1 "Conn_01x03_Male" H 8272 5073 50  0000 R CNN
 F 2 "Connector_JST:JST_XH_B3B-XH-A_1x03_P2.50mm_Vertical" H 8300 5050 50  0001 C CNN
@@
 $EndComp
 $Comp
-L power:+3.3V #PWR0107
+L power:+3.3V #PWR023
 U 1 1 5E66EFA3
 P 8100 4950
-F 0 "#PWR0107" H 8100 4800 50  0001 C CNN
+F 0 "#PWR023" H 8100 4800 50  0001 C CNN
 F 1 "+3.3V" H 8115 5123 50  0000 C CNN
 F 2 "" H 8100 4950 50  0001 C CNN
@@
 $EndComp
 $Comp
-L power:GND #PWR0108
+L power:GND #PWR024
 U 1 1 5E66EFA9
 P 8100 5150
-F 0 "#PWR0108" H 8100 4900 50  0001 C CNN
+F 0 "#PWR024" H 8100 4900 50  0001 C CNN
 F 1 "GND" H 8105 4977 50  0000 C CNN
 F 2 "" H 8100 5150 50  0001 C CNN

Commit message: soft update + pcb main try 1
Parts:
- removed C1, C3: 10µ, Capacitor_SMD:C_0805_2012Metric_Pad1.15x1.40mm_HandSolder, symbol Device:C
- removed C2: 22µf, Capacitor_SMD:C_0805_2012Metric_Pad1.15x1.40mm_HandSolder, symbol Device:C
- removed C4, C7, C8: 100n, Capacitor_SMD:C_0805_2012Metric_Pad1.15x1.40mm_HandSolder, symbol Device:C
- removed C5: 100nF, Capacitor_SMD:C_0805_2012Metric_Pad1.15x1.40mm_HandSolder, symbol Device:C
- removed C6: 4.7µ, Capacitor_SMD:C_0805_2012Metric_Pad1.15x1.40mm_HandSolder, symbol Device:C
- removed J1, J5: Conn_01x04_Male, Connector_JST:JST_XH_B4B-XH-A_1x04_P2.50mm_Vertical, symbol Connector:Conn_01x04_Male
- removed J2, J3, J6, J7: Conn_01x03_Male, Connector_JST:JST_XH_B3B-XH-A_1x03_P2.50mm_Vertical, symbol Connector:Conn_01x03_Male
- removed J4: Conn_01x12_Male, Connector_JST:JST_XH_B12B-XH-A_1x12_P2.50mm_Vertical, symbol Connector:Conn_01x12_Male
- removed L1: 2.2µH, Inductor_SMD:L_0805_2012Metric_Pad1.15x1.40mm_HandSolder, symbol Device:L
- removed R1: 100k, Resistor_SMD:R_0805_2012Metric_Pad1.15x1.40mm_HandSolder, symbol Device:R
- removed R2, R3, R4: 10k, Resistor_SMD:R_0805_2012Metric_Pad1.15x1.40mm_HandSolder, symbol Device:R
- removed SW1: SW_SPDT, Connector_PinHeader_2.54mm:PinHeader_1x03_P2.54mm_Vertical, symbol Switch:SW_SPDT
- removed SW2: SW_Push, Button_Switch_SMD:SW_SPST_PTS645, symbol Switch:SW_Push
- removed TP1, TP2, TP3: TestPoint, TestPoint:TestPoint_Pad_D2.0mm, symbol Connector:TestPoint
- removed U1: TPS62172DSG, Package_SON:WSON-8-1EP_2x2mm_P0.5mm_EP0.9x1.6mm_ThermalVias, symbol Regulator_Switching:TPS62172DSG
- removed U2: LIS2DHTR, Package_LGA:LGA-14_2x2mm_P0.35mm_LayoutBorder3x4y, symbol ent-rescue:LIS2DHTR-ian
- removed U3: STM32F030K6Tx, Package_QFP:LQFP-32_7x7mm_P0.8mm, symbol MCU_ST_STM32F0:STM32F030K6Tx
Connections:
- no-connect marks 7 -> 0
