File: kicad/ent/ent.kicad_pcb (KiCad board)
At the start: 2 copper layers, 28 parts, among them J1 Conn_01x04_Male, J2 Conn_01x03_Male, J3 Conn_01x03_Male, J4 Conn_01x12_Male, J5 Conn_01x04_Male, J6 Conn_01x03_Male, J7 Conn_01x03_Male, SW1 SW_SPDT, SW2 SW_Push, U1 TPS62172DSG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

Commit message: soft update + pcb main try 1
Parts:
- added C25: 10n, Capacitor_SMD:C_0805_2012Metric_Pad1.15x1.40mm_HandSolder, B.Cu at (123.5, 91.5)
- added C26: 1µ, Capacitor_SMD:C_0805_2012Metric_Pad1.15x1.40mm_HandSolder, B.Cu at (121.7, 91.5)
- added SW3: SW_Push, Button_Switch_SMD:SW_SPST_PTS645, F.Cu at (125.7, 84.8)
- added SW4: SW_SPST, Connector_JST:JST_XH_B2B-XH-A_1x02_P2.50mm_Vertical, F.Cu at (108.3, 111.9)
- C3, C4, C6, C7, C8: moved to B.Cu
- SW2: value SW_Push -> SW_SPST; footprint Button_Switch_SMD:SW_SPST_PTS645 -> Connector_JST:JST_XH_B2B-XH-A_1x02_P2.50mm_Vertical
- moved J4 54.2 mm to (145.1, 80.0), turned to 270 degrees
- moved J1 47.3 mm to (129.8, 73.3)
- moved C5 40.8 mm to (125.6, 90.9), turned to 180 degrees
- moved C8 40.3 mm to (129.1, 92.8)
- moved C6 38.4 mm to (122.9, 96.9), turned to 180 degrees
- moved J3 34.3 mm to (108.5, 80.3), turned to 270 degrees
- moved C1 32.3 mm to (137.2, 107.3), turned to 270 degrees
- moved J6 32.3 mm to (107.5, 73.2)
- moved J2 31.9 mm to (118.5, 73.2)
- moved R2 31.2 mm to (120.9, 105.0)
- moved L1 28.7 mm to (130.9, 105.1), turned to 180 degrees
- moved C4 27.3 mm to (117.2, 107.0), turned to 270 degrees
- moved SW2 25.3 mm to (108.3, 102.9), turned to 270 degrees
- moved C7 21.8 mm to (116.7, 101.2), turned to 180 degrees
- moved U1 20.6 mm to (134.5, 105.9), turned to 180 degrees
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Connections:
- SW2 pad 1: GND -> SW1
- SW2 pad 2: Net-(C5-Pad2) -> GND
- U3 pad 10: Net-(U3-Pad10) -> SW1
- U3 pad 11: Net-(U3-Pad11) -> SW2
- U3 pad 12: NSS3 -> NSS4
- U3 pad 13: NSS4 -> NSS3
- U3 pad 14: NSS1 -> NSS2
- U3 pad 15: NSS2 -> NSS1
Routing:
- net VOS: track 0.00 -> 66.6 mm, vias 0 -> 11
- net Net-(J1-Pad3): track 0.00 -> 50.2 mm, vias 0 -> 2
- net GND: track 0.00 -> 50.1 mm, vias 0 -> 5
- net Net-(J1-Pad2): track 0.00 -> 42.2 mm, vias 0 -> 2
- net NSS1: track 0.00 -> 30.8 mm, vias 0 -> 2
- net NSS4: track 0.00 -> 30.6 mm, vias 0 -> 1
- net NSS2: track 0.00 -> 29.8 mm, vias 0 -> 2
- net NSS3: track 0.00 -> 28.3 mm, vias 0 -> 1
- net STOP2: track 0.00 -> 24.2 mm
- net SPI1_MOSI: track 0.00 -> 24.1 mm
- net SPI1_MISO: track 0.00 -> 23.4 mm
- net SPI1_SCK: track 0.00 -> 22.7 mm
- net Net-(J4-Pad5): track 0.00 -> 22.0 mm
- net SW2: track 0.00 -> 21.3 mm
- net STOP1: track 0.00 -> 20.0 mm
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- added copper zone on B.Cu, net GND
- added copper zone on F.Cu, net VOS
Other:
- net class Default: clearance 0.2 -> 0.15
- rule trace_clearance: 0.2 -> 0.15
- rule trace_min: 0.2 -> 0.15

Commit message: pcb
Parts:
- added H1: MountingHole_Pad, MountingHole:MountingHole_3.2mm_M3_Pad, F.Cu at (102.0, 120.0)
- added H2: MountingHole_Pad, MountingHole:MountingHole_3.2mm_M3_Pad, F.Cu at (146.0, 67.0)
- added H3: MountingHole_Pad, MountingHole:MountingHole_3.2mm_M3_Pad, F.Cu at (146.0, 120.0)
- added H4: MountingHole_Pad, MountingHole:MountingHole_3.2mm_M3_Pad, F.Cu at (102.0, 67.0)
Routing:
- net GND: track 50.1 -> 49.7 mm, vias 5 -> 7
Other:
- board outline added: 52 x 61 mm
- net class Default: clearance 0.15 -> 0.16
- rule trace_clearance: 0.15 -> 0.16
- rule trace_min: 0.15 -> 0.16
