File: kicad/ent/ent.kicad_pcb (KiCad board)
At the start: 2 copper layers, 66 x 66 mm, 32 parts, among them J1 Conn_01x04_Male, J2 Conn_01x03_Male, J3 Conn_01x03_Male, J4 Conn_01x12_Male, J5 Conn_01x04_Male, J6 Conn_01x03_Male, J7 Conn_01x03_Male, SW1 SW_SPDT, SW2 SW_Push, SW3 SW_Push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

Commit message: pcb done
Parts:
- added D2: LED, LED_SMD:LED_0805_2012Metric_Pad1.15x1.40mm_HandSolder, F.Cu at (218.8, 81.0)
- added H1: MountingHole_Pad, MountingHole:MountingHole_2.2mm_M2_Pad, F.Cu at (169.5, 110.5)
- added H2: MountingHole_Pad, MountingHole:MountingHole_2.2mm_M2_Pad, F.Cu at (227.3, 109.9)
- added H3: MountingHole_Pad, MountingHole:MountingHole_2.2mm_M2_Pad, F.Cu at (227.3, 50.2)
- added H4: MountingHole_Pad, MountingHole:MountingHole_2.2mm_M2_Pad, F.Cu at (170.2, 50.2)
- added R7: R_Small, Resistor_SMD:R_0805_2012Metric_Pad1.15x1.40mm_HandSolder, F.Cu at (214.0, 81.1)
Connections:
- U3 pad 20: Net-(U3-Pad20) -> LED
Routing:
- net LED: track 0.00 -> 5.11 mm
- net Net-(D2-Pad2): track 0.00 -> 2.71 mm
- net GND: track 47.3 -> 49.2 mm, vias 7 -> 9
Other:
- board size 66 x 66 mm -> 66 x 68.6 mm

Commit message: software
functioneel
Parts:
- moved H4 1.27 mm to (168.9, 50.2)
- moved H1 0.63 mm to (168.9, 110.5)
Routing:
- net +12V: track 14.0 -> 28.0 mm
Other:
- outline, holes or cut-outs redrawn
Changed lines of the file:
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@@
     (thickness 1.6)
     (drawings 10)
-    (tracks 273)
+    (tracks 276)
     (zones 0)
     (modules 38)
@@
   )
   (module MountingHole:MountingHole_2.2mm_M2_Pad (layer F.Cu)
-    (at 169.545 110.49)
+    (at 168.91 110.49)
     (descr "Mounting Hole 2.2mm, M2")
     (tags "mounting hole 2.2mm m2")
@@
   )
   (module MountingHole:MountingHole_2.2mm_M2_Pad (layer F.Cu)
-    (at 170.18 50.165)
+    (at 168.91 50.165)
     (descr "Mounting Hole 2.2mm, M2")
     (tags "mounting hole 2.2mm m2")
@@
     )
   )
-  (gr_line (start 165.1 50.8) (end 165.1 110.49) (layer Edge.Cuts) (width 0.1))
+  (gr_line (start 165.1 49.53) (end 165.1 110.49) (layer Edge.Cuts) (width 0.1))
   (gr_line (start 231.14 110.49) (end 231.14 49.53) (layer Edge.Cuts) (width 0.1))
   (gr_arc (start 227.33 110.49) (end 227.33 114.3) (angle -90) (layer Edge.Cuts) (width 0.1))
   (gr_arc (start 168.91 110.49) (end 165.1 110.49) (angle -90) (layer Edge.Cuts) (width 0.1))
   (gr_arc (start 227.33 49.53) (end 231.14 49.53) (angle -90) (layer Edge.Cuts) (width 0.1))
-  (gr_arc (start 170.18 50.8) (end 170.18 45.72) (angle -90) (layer Edge.Cuts) (width 0.1))
+  (gr_arc (start 168.91 49.53) (end 168.91 45.72) (angle -90) (layer Edge.Cuts) (width 0.1))
   (dimension 66.04 (width 0.15) (layer Dwgs.User)
     (gr_text "66.040 mm" (at 234.726 81.28 270) (layer Dwgs.User)
@@
     (arrow2b (pts (xy 165.1 45.974) (xy 166.226504 45.387579)))
   )
-  (gr_line (start 227.33 45.72) (end 170.18 45.72) (layer Edge.Cuts) (width 0.1))
+  (gr_line (start 227.33 45.72) (end 168.91 45.72) (layer Edge.Cuts) (width 0.1))
   (gr_line (start 168.91 114.3) (end 227.33 114.3) (layer Edge.Cuts) (width 0.1))
   (segment (start 216.535 102.794264) (end 216.535 102.37) (width 0.25) (layer F.Cu) (net 1))
@@
   (segment (start 222.758 100.844885) (end 221.122885 102.48) (width 0.25) (layer F.Cu) (net 2))
   (segment (start 222.758 100.2792) (end 222.758 100.844885) (width 0.25) (layer F.Cu) (net 2))
+  (segment (start 225.4954 88.6378) (end 226.7204 88.6378) (width 0.25) (layer B.Cu) (net 2))
+  (segment (start 222.758 91.3752) (end 225.4954 88.6378) (width 0.25) (layer B.Cu) (net 2))
+  (segment (start 222.758 100.2792) (end 222.758 91.3752) (width 0.25) (layer B.Cu) (net 2))
   (via (at 213.995 106.68) (size 0.8) (drill 0.4) (layers F.Cu B.Cu) (net 3))
   (segment (start 213.995 102.235) (end 214.38 102.62) (width 0.25) (layer F.Cu) (net 3))
@@
     (polygon
       (pts
-        (xy 231.14 114.3) (xy 165.1 114.3) (xy 165.1 45.085) (xy 231.14 45.085)
+        (xy 231.14 114.3) (xy 162.56 114.3) (xy 162.56 45.085) (xy 231.14 45.085)
       )
     )
@@
     (polygon
       (pts
-        (xy 231.14 114.3) (xy 165.1 114.3) (xy 165.1 44.45) (xy 231.14 44.45)
+        (xy 231.14 114.3) (xy 163.83 114.3) (xy 163.83 44.45) (xy 231.14 44.45)
       )
     )
