File: kicad/ent/motor.kicad_pcb (KiCad board)
At the start: 2 copper layers, 99.9 x 78.7 mm, 28 parts, among them J10 Conn_01x02_Male, J11 Conn_01x02_Male, J12 Barrel_Jack, J13 Conn_01x12_Male, J14 Conn_01x12_Male, J8 Conn_01x02_Male, J9 Conn_01x02_Male, U4 IFX9201SGAUMA1, U5 IFX9201SGAUMA1, U6 IFX9201SGAUMA1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

Commit message: pcb
Parts:
- moved J13 60.0 mm to (115.4, 129.4), turned to 180 degrees
- moved J11 50.1 mm to (144.7, 79.7), turned to 90 degrees
- moved C13 48.9 mm to (141.4, 75.4), turned to 0 degrees
- moved C18 42.4 mm to (141.4, 84.3), turned to 0 degrees
- moved J10 37.2 mm to (144.6, 109.7), turned to 90 degrees
- moved U7 37.0 mm to (132.8, 79.5), turned to 90 degrees
- moved C17 36.0 mm to (141.3, 113.8), turned to 0 degrees
- moved C11 35.9 mm to (61.0, 124.4), turned to 180 degrees
- moved J8 35.9 mm to (57.3, 93.8), turned to 270 degrees
- moved C15 34.5 mm to (60.7, 89.6), turned to 180 degrees
- moved J9 34.4 mm to (57.6, 120.4), turned to 270 degrees
- moved C24 33.1 mm to (134.3, 86.4), turned to 0 degrees
- moved C14 32.3 mm to (68.6, 86.4), turned to 180 degrees
- moved C22 31.1 mm to (134.7, 117.2), turned to 0 degrees
- moved C21 31.0 mm to (133.1, 122.6)
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Connections:
- U4 pad 13: (no net) -> GND
- U5 pad 13: (no net) -> GND
- U6 pad 13: (no net) -> GND
- U7 pad 13: (no net) -> GND
Routing:
- net VOS: track 0.00 -> 249.3 mm
- net SPI1_MOSI: track 0.00 -> 189.4 mm, vias 0 -> 8
- net SPI1_SCK: track 0.00 -> 179.8 mm, vias 0 -> 9
- net SPI1_MISO: track 0.00 -> 179.7 mm, vias 0 -> 13
- net Net-(J14-Pad5): track 0.00 -> 176.5 mm, vias 0 -> 9
- net NSS2: track 0.00 -> 88.5 mm, vias 0 -> 2
- net +12V: track 90.3 -> 7.38 mm
- net PWM4: track 0.00 -> 69.9 mm, vias 0 -> 2
- net GND: track 2.53 -> 67.3 mm, vias 0 -> 48
- net NSS3: track 0.00 -> 59.7 mm, vias 0 -> 2
- net DIR1: track 0.00 -> 58.5 mm, vias 0 -> 3
- net NSS1: track 0.00 -> 56.8 mm, vias 0 -> 2
- net DIR4: track 0.00 -> 54.1 mm, vias 0 -> 4
- net PWM3: track 0.00 -> 46.1 mm, vias 0 -> 4
- net PWM1: track 0.00 -> 46.1 mm, vias 0 -> 4
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- added copper zone on F.Cu, net +12V
- added copper zone on B.Cu, net GND
- removed copper zone on B.Cu, net +12V
Other:
- net class Default: clearance 0.2 -> 0.15
- rule trace_clearance: 0.2 -> 0.15
